Commit message: 调整模型加载规则，实现多模型载入

File: assets/excavator_simple/excavator.urdf (robot description, URDF)
Before this commit: robot pudong, 17 links, 16 joints
Links:
- removed link base_link
- removed link chandou
- removed link cheshen
- removed link pjjq03
- removed link pjjq04
- removed link pjjq05_1
- removed link pjjq05_2
- removed link pjjq06
- removed link yg1050
- removed link yg1050_2
- removed link yg1220_1_1
- removed link yg1220_1_2
- removed link yg1220_2_1
- removed link yg1220_2_2
- removed link yg1480
- removed link yg1480_2
- added link 10_bucket_rocker_left, mass 3.6933; collision mesh filename=package://excavator/meshes/10_bucket_rocker_left.STL; visual mesh filename=package://excavator/meshes/10_bucket_rocker_left.STL
- added link 10_bucket_rocker_right, mass 3.6933; collision mesh filename=package://excavator/meshes/10_bucket_rocker_right.STL; visual mesh filename=package://excavator/meshes/10_bucket_rocker_right.STL
- added link 11_bucket_link, mass 16.973; collision mesh filename=package://excavator/meshes/11_bucket_link.STL; visual mesh filename=package://excavator/meshes/11_bucket_link.STL
- added link 1_base, mass 2592.7; collision mesh filename=package://excavator/meshes/1_base.STL; visual mesh filename=package://excavator/meshes/1_base.STL
- added link 2_swing, mass 7793.2; collision mesh filename=package://excavator/meshes/2_swing.STL; visual mesh filename=package://excavator/meshes/2_swing.STL
- added link 3_boom, mass 1440.8; collision mesh filename=package://excavator/meshes/3_boom.STL; visual mesh filename=package://excavator/meshes/3_boom.STL
- added link 4_boom_cylinder_left_down, mass 12.766; collision mesh filename=package://excavator/meshes/4_boom_cylinder_left_down.STL; visual mesh filename=package://excavator/meshes/4_boom_cylinder_left_down.STL
- added link 4_boom_cylinder_left_up, mass 8.7504; collision mesh filename=package://excavator/meshes/4_boom_cylinder_left_up.STL; visual mesh filename=package://excavator/meshes/4_boom_cylinder_left_up.STL
- added link 5_boom_cylinder_right_down, mass 12.766; collision mesh filename=package://excavator/meshes/5_boom_cylinder_right_down.STL; visual mesh filename=package://excavator/meshes/5_boom_cylinder_right_down.STL
- added link 5_boom_cylinder_right_up, mass 8.7504; collision mesh filename=package://excavator/meshes/5_boom_cylinder_right_up.STL; visual mesh filename=package://excavator/meshes/5_boom_cylinder_right_up.STL
- added link 6_stick, mass 600.4; collision mesh filename=package://excavator/meshes/6_stick.STL; visual mesh filename=package://excavator/meshes/6_stick.STL
- added link 7_stick_cylinder_down, mass 15.576; collision mesh filename=package://excavator/meshes/7_stick_cylinder_down.STL; visual mesh filename=package://excavator/meshes/7_stick_cylinder_down.STL
- added link 7_stick_cylinder_up, mass 15.423; collision mesh filename=package://excavator/meshes/7_stick_cylinder_up.STL; visual mesh filename=package://excavator/meshes/7_stick_cylinder_up.STL
- added link 8_bucket, mass 359.5; collision mesh filename=package://excavator/meshes/8_bucket.STL; visual mesh filename=package://excavator/meshes/8_bucket.STL
- added link 9_bucket_cylinder_down, mass 11.684; collision mesh filename=package://excavator/meshes/9_bucket_cylinder_down.STL; visual mesh filename=package://excavator/meshes/9_bucket_cylinder_down.STL
- added link 9_bucket_cylinder_up, mass 8.1381; collision mesh filename=package://excavator/meshes/9_bucket_cylinder_up.STL; visual mesh filename=package://excavator/meshes/9_bucket_cylinder_up.STL
Joints:
- joint 03_to_04: child pjjq04 -> 6_stick; parent pjjq03 -> 3_boom
- joint 03_to_1480: child yg1480 -> 7_stick_cylinder_down; parent pjjq03 -> 3_boom
- joint 04_to_05_1: child pjjq05_1 -> 10_bucket_rocker_left; parent pjjq04 -> 6_stick
- joint 04_to_05_2: child pjjq05_2 -> 10_bucket_rocker_right; parent pjjq04 -> 6_stick
- joint 04_to_1050: child yg1050 -> 9_bucket_cylinder_down; parent pjjq04 -> 6_stick
- joint 04_to_chandou: child chandou -> 8_bucket; parent pjjq04 -> 6_stick
- joint 1050_1_to_2: child yg1050_2 -> 9_bucket_cylinder_up; parent yg1050 -> 9_bucket_cylinder_down
- joint 1220_1: child yg1220_1_2 -> 4_boom_cylinder_left_up; parent yg1220_1_1 -> 4_boom_cylinder_left_down
- joint 1220_2: child yg1220_2_2 -> 5_boom_cylinder_right_up; parent yg1220_2_1 -> 5_boom_cylinder_right_down
- joint 1480_1_to_2: child yg1480_2 -> 7_stick_cylinder_up; parent yg1480 -> 7_stick_cylinder_down
- joint base_footprint_joint: child base_link -> 1_base
- joint base_to_cheshen: child cheshen -> 2_swing; parent base_link -> 1_base
- joint chandou_to_06: child pjjq06 -> 11_bucket_link; parent chandou -> 8_bucket
- joint cheshen_to_03: child pjjq03 -> 3_boom; parent cheshen -> 2_swing
- joint cheshen_to_1220_1: child yg1220_1_1 -> 4_boom_cylinder_left_down; parent cheshen -> 2_swing
- joint cheshen_to_1220_2: child yg1220_2_1 -> 5_boom_cylinder_right_down; parent cheshen -> 2_swing

Commit message: 优化项目结构

File: assets/excavator_simple/excavator.urdf (robot description, URDF)
Before this commit: robot excavator, 17 links, 16 joints
Links:
- removed link 10_bucket_rocker_left
- removed link 10_bucket_rocker_right
- removed link 11_bucket_link
- removed link 4_boom_cylinder_left_down
- removed link 4_boom_cylinder_left_up
- removed link 5_boom_cylinder_right_down
- removed link 5_boom_cylinder_right_up
- removed link 7_stick_cylinder_down
- removed link 7_stick_cylinder_up
- removed link 9_bucket_cylinder_down
- removed link 9_bucket_cylinder_up
Joints:
- removed joint 03_to_04
- removed joint 03_to_1480
- removed joint 04_to_05_1
- removed joint 04_to_05_2
- removed joint 04_to_1050
- removed joint 04_to_chandou
- removed joint 1050_1_to_2
- removed joint 1220_1
- removed joint 1220_2
- removed joint 1480_1_to_2
- removed joint base_to_cheshen
- removed joint chandou_to_06
- removed joint cheshen_to_03
- removed joint cheshen_to_1220_1
- removed joint cheshen_to_1220_2
- added joint j1_swing: type continuous, parent 1_base, child 2_swing, origin xyz=0 0 0.72 rpy=0 0 0, axis 0 0 -1
- added joint j2_boom: type revolute, parent 2_swing, child 3_boom, origin xyz=-0.009 0 1.0372 rpy=0 0 0, axis 0 1 0, limit lower=-0.9 upper=0.3 effort=0 velocity=1
- added joint j3_stick: type revolute, parent 3_boom, child 6_stick, origin xyz=5.4177 0 1.706 rpy=0 1.2726 0, axis 0 1 0, limit lower=-0.8 upper=1.0 effort=0 velocity=1
- added joint j4_bucket: type revolute, parent 6_stick, child 8_bucket, origin xyz=2.9111 0 0.15097 rpy=0 1.4717 0, axis 0 1 0, limit lower=-2.1 upper=0.6 effort=0 velocity=1
