Commit message: 实现挖一斗

File: assets/excavator_s010/excavator.urdf (robot description, URDF)
Before this commit: robot excavator, 6 links, 5 joints
Links:
- link 8_bucket: geometry collision box size=0.010 0.086 0.060; collision box size=0.010 0.086 0.060

Commit message: 完善环境

File: assets/excavator_s010/excavator.urdf (robot description, URDF)
Before this commit: robot excavator, 6 links, 5 joints
Links:
- link 8_bucket: geometry collision box size=0.002 0.086 0.060; collision box size=0.010 0.086 0.060
